File: alt-panel/alt-panel.kicad_pcb (KiCad board)
At the start: 2 copper layers, 91.3 x 128.5 mm, 31 parts

Commit message: Panel tweak
Parts:
- moved REF** 0.55 mm to (62.8, 100.0)
- moved REF** 0.50 mm to (62.8, 65.0)
- moved REF** 0.45 mm to (62.8, 29.5)
- moved REF** 0.30 mm to (29.2, 30.2)
- moved REF** 0.25 mm to (38.0, 126.5)
- moved REF** 0.25 mm to (34.0, 126.4)
- moved REF** 0.25 mm to (50.8, 126.5)
- moved REF** 0.25 mm to (29.2, 65.8)
- moved REF** 0.20 mm to (29.2, 100.8)

Commit message: Panel tweaks
Parts:
- moved REF** 0.65 mm to (85.2, 91.2)
- moved REF** 0.50 mm to (85.2, 107.8)
- moved REF** 0.50 mm to (85.2, 72.8)
- moved REF** 0.50 mm to (8.00, 107.8)
- moved REF** 0.50 mm to (6.25, 91.2)
- moved REF** 0.50 mm to (8.00, 37.2)
- moved REF** 0.50 mm to (6.25, 56.1)
- moved REF** 0.50 mm to (85.2, 56.2)
- moved REF** 0.50 mm to (85.2, 37.2)
- moved REF** 0.50 mm to (8.00, 72.8)
- moved REF** 0.50 mm to (85.2, 20.7)
- moved REF** 0.50 mm to (6.25, 20.7)
Other:
- outline, holes or cut-outs redrawn
