File: mainboard/mainboard.kicad_sch (KiCad schematic)
At the start: 126 parts, among them J1 Eurorack_Power, J10 H2, J11 CV3, J12 O3, J13 H3, J2 R1, J3 CV1, J4 R2, J5 O1, J6 H1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

Commit message: Some more routing, moved D2, D5 and D8 to make it cleanr
Parts:
- U2: value 40106 -> (none); footprint Package_DIP:DIP-14_W7.62mm_Socket -> (none)
Connections:
- net CmpVref: now also U6.13 (-), U6.2 (-), U6.6 (-), U6.7, U6.9 (-); no longer U6.1, U6.13 (-), U6.2 (-), U6.6 (-), U6.9 (-)
- net Out1: now also U2.8, U3.4; no longer U2.4, U3.1
- net Out2: now also U2.12, U3.8; no longer U2.8, U3.4
- net Out3: now also U2.10, U3.1; no longer U2.12, U3.8
- net R1o: now also U3.5, U6.1; no longer U3.13, U6.7
- net R2o: now also U3.6, U6.14; no longer U3.5, U6.8
- net R3o: now also U3.13, U6.8; no longer U3.6, U6.14
- net Vref: now also U4.13 (-), U4.14, U4.2 (-), U4.6 (-), U4.9 (-); no longer U4.1, U4.13 (-), U4.2 (-), U4.6 (-), U4.9 (-)
- net at R32.2, U7.1 (CP): now also U3.9; no longer U3.3
- net at D5.1 (K), R34.2, SW2.2 (B): now also U2.3; no longer U2.5
- net at C11.1, D5.2 (A): now also U2.4; no longer U2.6
- net at C11.2, R31.2: now also U4.3 (+); no longer U4.10 (+)
- net at C15.2, R48.2: now also U4.5 (+); no longer U4.12 (+)
- net at D11.1 (K), R7.2: now also U6.3 (+); no longer U6.5 (+)
- net at C8.2, R12.2: now also U4.10 (+); no longer U4.5 (+)
- net at D2.1 (K), R15.2, SW1.2 (B): now also U2.5; no longer U2.1
- net at C8.1, D2.2 (A): now also U2.6; no longer U2.2
- net at R13.2, U7.9 (CP): now also U3.3; no longer U3.2
- net at D8.1 (K), R51.2, SW3.2 (B): now also U2.1; no longer U2.11
- net at C15.1, D8.2 (A): now also U2.2; no longer U2.10
- net at D13.1 (K), R26.2: now also U6.10 (+); no longer U6.12 (+)
- net at R49.2, U8.1 (CP), U8.9 (CP): now also U3.2; no longer U3.9
- net at R3.2, R6.1: now also U6.5 (+); no longer U6.3 (+)
- net at C5.1, R1.2, R4.1: now also U4.12 (+); no longer U4.3 (+)
- net at D12.1 (K), R22.2: now also U6.12 (+); no longer U6.10 (+)
- new net: U2.9, U4.8
- new net: U2.11, U4.7
- new net: U2.13, U4.1
Other:
- title: (none) -> GrassiOsc

Commit message: Routing
Parts:
- removed D10, D11, D12, D13, D4, D7: 1N4148, Diode_THT:D_DO-35_SOD27_P7.62mm_Horizontal, symbol Device:D
- added D10, D11, D12, D13, D4, D7: BAT85, Diode_THT:D_DO-35_SOD27_P7.62mm_Horizontal, symbol Diode:BAT85
- U2: value (none) -> 40106; footprint (none) -> Package_DIP:DIP-14_W7.62mm_Socket
- U6: value TL074 -> LM324
Connections:
- net GND: now also D10.2 (A), D11.2 (A), D12.2 (A), D13.2 (A), D4.2 (A), D7.2 (A)
- net Hav3: now also U5.1; no longer U5.14
- net Vref2: now also U5.13 (-), U5.14, U5.3 (+); no longer U5.1, U5.12 (+), U5.2 (-)
- net at R44.1, R56.2, R57.2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: now also U5.2 (-); no longer U5.13 (-)
- net at R7.2, U6.3 (+): now also D11.1 (K)
- net at Q4.2 (B), R29.2, R33.2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: now also D7.1 (K)
- net at Q6.2 (B), R46.2, R50.2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: now also D10.1 (K)
- net at R26.2, U6.10 (+): now also D13.1 (K)
- net at C6.1, R2.2, R5.1: now also U5.12 (+); no longer U5.3 (+)
- net at Q2.2 (B), R10.2, R14.2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: now also D4.1 (K)
- net at R22.2, U6.12 (+): now also D12.1 (K)

Commit message: Rerouted: number of vias reduced from 39 to 13
Connections:
- net Hav1: now also J6.T, R21.2; no longer R21.1, R8.2, R9.1, U5.7
- net Hav2: now also J10.T, R40.2; no longer R27.2, R28.1, R40.1, U5.8
- net Hav3: now also J13.T, R53.2; no longer R44.2, R45.1, R53.1, U5.1
- net at D5.1 (K), R34.2, SW2.2 (B)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: now also C11.1
- net at D5.2 (A), U2.4: no longer C11.1
- net at D2.1 (K), R15.2, SW1.2 (B)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: now also C8.1
- net at D2.2 (A), U2.6: no longer C8.1
- net at D8.1 (K), R51.2, SW3.2 (B)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: now also C15.1
- net at D8.2 (A), U2.2: no longer C15.1
- new net: R21.1, R8.2, R9.1, U5.7
- new net: R44.2, R45.1, R53.1, U5.1
- new net: R27.2, R28.1, R40.1, U5.8
Other:
- moved on the sheet: C11, C15, C8, J12, J5, J9, R12, R20, R21, R31, R37, R40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
